File: PCB/macropad.kicad_pcb (KiCad board)
At the start: 2 copper layers, 61.9 x 64.3 mm, 10 parts, among them J1 I2C_Connector, SW1 SW_Push, SW2 SW_Push, SW3 SW_Push, SW4 SW_Push, SW5 SW_Push, SW6 SW_Push, U1 XIAO-RP2040-DIP

Commit message: image and schematic updates
Parts:
- removed R1: 400Ω, Resistor:R_Axial_DIN0204_L3.6mm_D1.6mm_P5.08mm_Horizontal
Connections:
- U1 pad 3: Net-(U1-GPIO28/ADC2/A2) -> Net-(D2-DIN)
Routing:
- net Net-(D2-DIN): track 15.3 -> 43.2 mm, vias 1 -> 2
- net Net-(U1-GPIO28/ADC2/A2): track 24.1 -> 0.00 mm
